File: esp32.kicad_sch (KiCad schematic)
At the start: 14 parts, among them Q1 2N5088BU_Obsolete, Q2 2N5088BU_Obsolete, U6 MCP6002-I_P, U7 MCP6002-I_P

Commit message: wip on esp conns
Parts:
- added C40, C41: 22uF, symbol Device:C
- added D2: SS34, Diode_SMD:D_SMA, symbol Diode:SS34
- added D3: LED_ABGR, symbol Device:LED_ABGR
- added J2, J3: 0022232041, digikey-footprints:PinHeader_1x4_P2.54mm_Drill1.02mm, symbol dk_Rectangular-Connectors-Headers-Male-Pins:0022232041
- added J5: 640456-2, digikey-footprints:PinHeader_1x2_P2.54mm_Drill1.02mm, symbol dk_Rectangular-Connectors-Headers-Male-Pins:640456-2
- added L2: 22uH, symbol Device:L
- added R4: 2k_0603, 4ms_Resistor:R_0603, symbol PCM_4ms_Resistor:2k_0603
- added R5: 150R_0603, 4ms_Resistor:R_0603, symbol PCM_4ms_Resistor:150R_0603
- added U2: MT3608, Package_TO_SOT_SMD:SOT-23-6, symbol Regulator_Switching:MT3608
Connections:
- net GNDD: now also A2.4 (GND), C40.2, C41.2, D3.1 (A), J2.1, R5.2, U2.2 (GND)
- net PWM0: now also A2.20 (A7/IO32)
- net PWM1: now also A2.22 (A9/IO33)
- net U4B: now also A2.5 (DAC2/A0)
- net U4D: now also A2.6 (DAC1/A1)
- net RESET: now reaches A2.1 (~{RESET})
- net at A2.14 (RX/IO16): now also D3.2 (BK)
- net at A2.15 (TX/IO17): now also D3.3 (GK)
- net at A2.16 (IO21): now also D3.4 (RK)
- net +3V3: now reaches A2.2 (3V3)
- net +3V3: now also C40.1, J2.4, L2.1, U2.4 (EN), U2.5 (IN)
- new net: D2.2 (A), L2.2, U2.1 (SW)
- new net: R4.2, R5.1, U2.3 (FB)
- new net +9V: C41.1, D2.1 (K), J3.4, R4.1
- new net AUDIO_IN: J3.2
- new net EFFECT_OUT: J3.3
- new net GNDA: J3.1
Other:
- note added: "LED to be used for determine effect 'state'"
- note added: "Power Supply"
- note added: "TODO: - adjustable gain for input OpAmp? - check caps. Maybe make components so better sizes? (learn to model) - vet the cap's ripple current. Assume ok for now - add connectors to breakout signals"
- note added: "boost converter considerations: - effiency (9V @ 500mA => 5V @ 1.1A) - expected current load (600 mA max?) - noise and ripple - as long as current ripple <RMS of caps :) - picked 10uH inductor. should b overkill - schottky diode. Consider forward V drop, reverse voltage rating, forward I rating, switching speed - 10k resistors enough for CC1 CC2??"
- moved on the sheet: A2

Commit message: fixed a lot of things
Other:
- note added: "add encoder add push buttons"
Changed lines of the file:
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@@
+		)
+	)
+	(text "add encoder\nadd push buttons\n"
+		(exclude_from_sim no)
+		(at 132.588 73.66 0)
+		(effects
+			(font
+				(size 1.27 1.27)
+			)
 		)
 	)
